File: hardware/industrial-digital-in-4-v2.kicad_pcb (KiCad board)
At the start: 2 copper layers, 40 x 40 mm, 34 parts, among them P1 CON-SENSOR2, P2 DEBUG, P3 BOOT, P4 Digital Input, U1 XMC1100, U2 LTV846S, U3 DRILL, U4 DRILL, U5 DRILL, U6 DRILL

Commit message: Change LED color
Parts:
- D2, D3, D4, D5: value green -> blue
Connections:
- P1 pad 1: (no net) -> Net-(P1-Pad1)
- U1 pad 11: (no net) -> Net-(U1-Pad11)
- U1 pad 12: (no net) -> Net-(U1-Pad12)
- U1 pad 17: (no net) -> Net-(U1-Pad17)
- U1 pad 19: (no net) -> Net-(U1-Pad19)
- U1 pad 2: (no net) -> Net-(U1-Pad2)
- U1 pad 20: (no net) -> Net-(U1-Pad20)
- U1 pad 8: (no net) -> Net-(U1-Pad8)
Changed lines of the file:
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@@
-(kicad_pcb (version 4) (host pcbnew 4.0.7-e2-6376~58~ubuntu17.04.1)
+(kicad_pcb (version 4) (host pcbnew 4.0.2+dfsg1-stable)
   (general
     (links 73)
     (no_connects 0)
-    (area 96.944659 37.196239 283.24585 163.390793)
+    (area 97.609659 37.858699 137.993121 78.242161)
     (thickness 1.6002)
     (drawings 34)
@@
     (zones 0)
     (modules 34)
-    (nets 39)
+    (nets 47)
   )
   (page A4)
@@
   (net 37 LED1)
   (net 38 LED0)
+  (net 39 "Net-(P1-Pad1)")
+  (net 40 "Net-(U1-Pad2)")
+  (net 41 "Net-(U1-Pad8)")
+  (net 42 "Net-(U1-Pad11)")
+  (net 43 "Net-(U1-Pad12)")
+  (net 44 "Net-(U1-Pad17)")
+  (net 45 "Net-(U1-Pad19)")
+  (net 46 "Net-(U1-Pad20)")
   (net_class Default "This is the default net class."
     (clearance 0.14986)
@@
     (add_net "Net-(D4-Pad2)")
     (add_net "Net-(D5-Pad2)")
+    (add_net "Net-(P1-Pad1)")
     (add_net "Net-(P1-Pad4)")
     (add_net "Net-(P1-Pad5)")
@@
     (add_net "Net-(R4-Pad1)")
     (add_net "Net-(R5-Pad1)")
+    (add_net "Net-(U1-Pad11)")
+    (add_net "Net-(U1-Pad12)")
+    (add_net "Net-(U1-Pad17)")
+    (add_net "Net-(U1-Pad19)")
+    (add_net "Net-(U1-Pad2)")
+    (add_net "Net-(U1-Pad20)")
+    (add_net "Net-(U1-Pad8)")
     (add_net S-CLK)
     (add_net S-CS)
@@
       (effects (font (size 0.2 0.2) (thickness 0.05)))
     )
-    (fp_text value green (at 0.75 0.45 270) (layer F.Fab)
+    (fp_text value blue (at 0.75 0.45 270) (layer F.Fab)
       (effects (font (size 0.2 0.2) (thickness 0.05)))
     )
@@
       (effects (font (size 0.2 0.2) (thickness 0.05)))
     )
-    (fp_text value green (at 0.75 0.45 270) (layer F.Fab)
+    (fp_text value blue (at 0.75 0.45 270) (layer F.Fab)
       (effects (font (size 0.2 0.2) (thickness 0.05)))
     )
@@
       (effects (font (size 0.2 0.2) (thickness 0.05)))
     )
-    (fp_text value green (at 0.75 0.45 270) (layer F.Fab)
+    (fp_text value blue (at 0.75 0.45 270) (layer F.Fab)
       (effects (font (size 0.2 0.2) (thickness 0.05)))
     )
@@
       (effects (font (size 0.2 0.2) (thickness 0.05)))
     )
-    (fp_text value green (at 0.75 0.45 270) (layer F.Fab)
+    (fp_text value blue (at 0.75 0.45 270) (layer F.Fab)
       (effects (font (size 0.2 0.2) (thickness 0.05)))
     )
@@
     (fp_line (start 6 -4.3) (end -6 -4.3) (layer F.Fab) (width 0.05))
     (fp_line (start -6 -4.3) (end -6 -0.25) (layer F.Fab) (width 0.05))
-    (pad 1 smd rect (at -3.75 -4.6 180) (size 0.6 1.8) (layers Front F.Paste F.Mask))
+    (pad 1 smd rect (at -3.75 -4.6 180) (size 0.6 1.8) (layers Front F.Paste F.Mask)
+      (net 39 "Net-(P1-Pad1)"))
     (pad 2 smd rect (at -2.5 -4.6 180) (size 0.6 1.8) (layers Front F.Paste F.Mask)
       (net 2 GND))
@@
     (pad 1 smd oval (at -2.025 -1.25) (size 1 0.3) (layers Front F.Paste F.Mask)
       (net 31 S-MISO))
-    (pad 2 smd oval (at -2.025 -0.75) (size 1 0.3) (layers Front F.Paste F.Mask))
+    (pad 2 smd oval (at -2.025 -0.75) (size 1 0.3) (layers Front F.Paste F.Mask)
+      (net 40 "Net-(U1-Pad2)"))
     (pad 3 smd oval (at -2.025 -0.25) (size 1 0.3) (layers Front F.Paste F.Mask)
       (net 3 INPUT1))
@@
     (pad 7 smd oval (at -1.25 2.025 90) (size 1 0.3) (layers Front F.Paste F.Mask)
       (net 21 "Net-(P3-Pad2)"))
-    (pad 8 smd oval (at -0.75 2.025 90) (size 1 0.3) (layers Front F.Paste F.Mask))
+    (pad 8 smd oval (at -0.75 2.025 90) (size 1 0.3) (layers Front F.Paste F.Mask)
+      (net 41 "Net-(U1-Pad8)"))
     (pad 9 smd oval (at -0.25 2.025 90) (size 1 0.3) (layers Front F.Paste F.Mask)
       (net 2 GND))
     (pad 10 smd oval (at 0.25 2.025 90) (size 1 0.3) (layers Front F.Paste F.Mask)
       (net 1 3V3))
-    (pad 11 smd oval (at 0.75 2.025 90) (size 1 0.3) (layers Front F.Paste F.Mask))
-    (pad 12 smd oval (at 1.25 2.025 90) (size 1 0.3) (layers Front F.Paste F.Mask))
+    (pad 11 smd oval (at 0.75 2.025 90) (size 1 0.3) (layers Front F.Paste F.Mask)
+      (net 42 "Net-(U1-Pad11)"))
+    (pad 12 smd oval (at 1.25 2.025 90) (size 1 0.3) (layers Front F.Paste F.Mask)
+      (net 43 "Net-(U1-Pad12)"))
     (pad 13 smd oval (at 2.025 1.25) (size 1 0.3) (layers Front F.Paste F.Mask)
       (net 35 LED3))
@@
     (pad 16 smd oval (at 2.025 -0.25) (size 1 0.3) (layers Front F.Paste F.Mask)
       (net 38 LED0))
-    (pad 17 smd oval (at 2.025 -0.75) (size 1 0.3) (layers Front F.Paste F.Mask))
+    (pad 17 smd oval (at 2.025 -0.75) (size 1 0.3) (layers Front F.Paste F.Mask)
+      (net 44 "Net-(U1-Pad17)"))
     (pad 18 smd oval (at 2.025 -1.25) (size 1 0.3) (layers Front F.Paste F.Mask)
       (net 10 "Net-(P2-Pad1)"))
-    (pad 19 smd oval (at 1.25 -2.025 90) (size 1 0.3) (layers Front F.Paste F.Mask))
-    (pad 20 smd oval (at 0.75 -2.025 90) (size 1 0.3) (layers Front F.Paste F.Mask))
+    (pad 19 smd oval (at 1.25 -2.025 90) (size 1 0.3) (layers Front F.Paste F.Mask)
+      (net 45 "Net-(U1-Pad19)"))
+    (pad 20 smd oval (at 0.75 -2.025 90) (size 1 0.3) (layers Front F.Paste F.Mask)
+      (net 46 "Net-(U1-Pad20)"))
     (pad 21 smd oval (at 0.25 -2.025 90) (size 1 0.3) (layers Front F.Paste F.Mask)
       (net 11 "Net-(R1-Pad1)"))

Commit message: Change capacitor footprint(s) to C0402F
Parts:
- C1: footprint C0805 -> kicad-libraries:C0805
- C2: footprint C0402E -> kicad-libraries:C0402F
- C3, C4: footprint C0603F -> kicad-libraries:C0603F
- D1, D2, D3, D4, D5: footprint D0603F -> kicad-libraries:D0603F
- P1: footprint CON-SENSOR2 -> kicad-libraries:CON-SENSOR2
- P4: footprint OQ_8P -> kicad-libraries:OQ_8P
- R1: footprint R0603F -> kicad-libraries:R0603F
- R2, R3, R4, R5: footprint R1210 -> kicad-libraries:R1210
- RP1: footprint 4X0402 -> kicad-libraries:4X0402
- RP2, RP3: footprint 0603X4 -> kicad-libraries:0603X4
- U2: footprint OPTO-SMD16 -> kicad-libraries:OPTO-SMD16
- U3, U4, U5, U6: footprint DRILL_NP -> kicad-libraries:DRILL_NP
