File: hardware/industrial-digital-in-4-v2.kicad_pcb (KiCad board)
At the start: 2 copper layers, 40 x 40 mm, 34 parts, among them P1 CON-SENSOR2, P2 DEBUG, P3 BOOT, P4 Digital Input, U1 XMC1100, U2 LTV846S, U3 DRILL, U4 DRILL, U5 DRILL, U6 DRILL

Commit message: Data Cleanup
Parts:
- moved U6 2.94 mm to (102.5, 77.5)
- moved P1 2.94 mm to (120.0, 40.0)
- moved D2 2.94 mm to (128.5, 42.5)
- moved G*** 2.94 mm to (130.0, 60.0)
- moved C1 2.94 mm to (122.0, 46.5)
- moved C3 2.94 mm to (118.8, 46.6)
- moved C4 2.94 mm to (105.8, 51.5)
- moved D1 2.94 mm to (111.5, 42.5)
- moved D3 2.94 mm to (130.1, 42.5)
- moved D4 2.94 mm to (131.7, 42.5)
- moved D5 2.94 mm to (133.3, 42.5)
- moved P3 2.94 mm to (102.8, 51.0)
- moved P4 2.94 mm to (120.0, 72.0)
- moved R1 2.94 mm to (110.1, 42.5)
- moved R2 2.94 mm to (107.7, 64.4)
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Other:
- net class Default removed
- board text added: "Copyright Tinkerforge GmbH 2023. This documentation describes Open Hardware and is licensed under the CERN OHL v. 1.1. You may redistribute and modify this documentation under the terms of the CERN OHL v.1.1. (http://ohwr.org/cernohl). This documentation is distributed WITHOUT ANY EXPRESS OR IMPLIED WARRANTY, INCLUDING OF MERCHANTABILITY, SATISFACTORY QUALITY AND FITNESS FOR A PARTICULAR PURPOSE.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"
- board text removed: "Copyright Tinkerforge GmbH 2018. This documentation describes Open Hardware and is licensed under the CERN OHL v. 1.1. You may redistribute and modify this documentation under the terms of the CERN OHL v.1.1. (http://ohwr.org/cernohl). This documentation is distributed WITHOUT ANY EXPRESS OR IMPLIED WARRANTY, INCLUDING OF MERCHANTABILITY, SATISFACTORY QUALITY AND FITNESS FOR A PARTICULAR PURPOSE.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"
